File: pcb/starbie_kicad_pcb/starbie_kicad_pcb.kicad_sch (KiCad schematic)
At the start: 6 parts, among them J1 Conn_01x04_Pin, J2 Conn_01x08_Pin, SW1 SW_Push, SW2 SW_Push, U1 XIAO-ESP32-C3-SMD, U2 DHT11

Commit message: updates from project for pcb
Parts:
- added R1: 10k, Resistor_THT:R_Axial_DIN0204_L3.6mm_D1.6mm_P7.62mm_Horizontal, symbol Device:R
- J1: footprint (none) -> starbie footprints:Display_128x64_096_I2C
- J2: footprint (none) -> Connector_PinHeader_2.54mm:PinHeader_1x08_P2.54mm_Vertical
- SW1, SW2: footprint (none) -> Button_Switch_Keyboard:SW_Cherry_MX_1.00u_PCB
- U2: renamed from U1; footprint Seeed_Studio_XIAO_Series:XIAO-ESP32-C3-SMD -> starbie footprints:XIAO-ESP32-C6-DIP
- renumbered U2 to U1
Connections:
- net +3.3V: now also U1.1 (VDD), R1.1
- net DHT11 DATA: now also U1.2 (DATA), R1.2
- net GND: now also U1.4 (GND)
Other:
- note added: "ENVIRONMENT SENSOR"
- moved on the sheet: U1

Commit message: added arduino sketch files
Connections:
- net +3.3V: now also J1.2 (Pin_2)
- net GND: now also J1.1 (Pin_1)
- net SCL: now also J1.3 (Pin_3)
- net SDA: now also J1.4 (Pin_4)
Changed lines of the file:
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@@
+	(wire
+		(pts
+			(xy 146.05 137.16) (xy 146.05 133.35)
+		)
+		(stroke
+			(width 0)
+			(type default)
+		)
+	)
 	(wire
 		(pts
@@
 	(wire
 		(pts
+			(xy 156.21 137.16) (xy 146.05 137.16)
+		)
+		(stroke
+			(width 0)
+			(type default)
+		)
+	)
+	(wire
+		(pts
+			(xy 156.21 129.54) (xy 156.21 137.16)
+		)
+		(stroke
+			(width 0)
+			(type default)
+		)
+	)
+	(wire
+		(pts
 			(xy 186.69 119.38) (xy 187.96 119.38)
 		)
@@
 	(wire
 		(pts
+			(xy 158.75 129.54) (xy 158.75 132.08)
+		)
+		(stroke
+			(width 0)
+			(type default)
+		)
+	)
+	(wire
+		(pts
 			(xy 127 146.05) (xy 127 147.32)
 		)
@@
 	(wire
 		(pts
+			(xy 153.67 129.54) (xy 153.67 132.08)
+		)
+		(stroke
+			(width 0)
+			(type default)
+		)
+	)
+	(wire
+		(pts
 			(xy 166.37 83.82) (xy 166.37 86.36)
 		)
@@
 		(pts
 			(xy 163.83 83.82) (xy 166.37 83.82)
+		)
+		(stroke
+			(width 0)
+			(type default)
+		)
+	)
+	(wire
+		(pts
+			(xy 151.13 129.54) (xy 151.13 132.08)
 		)
 		(stroke
@@
 	)
 	(label "SCL"
-		(at 151.13 132.08 270)
+		(at 153.67 132.08 270)
 		(effects
 			(font
@@
 	)
 	(label "SDA"
-		(at 153.67 132.08 270)
-		(effects
-			(font
+		(at 151.13 132.08 270)
+		(effects
+			(font
